Commit message: PartA mostly done

File: nuturtle_description/urdf/turtlebot3_burger.urdf.xacro (robot description, xacro)
@@ -6,11 +6,13 @@
   <xacro:property name="wheel_radius" value="${param['wheel_radius']}" />
   <xacro:property name="track_width" value="${param['track_width']}" />
-  <link name="base_footprint"/>
-  <joint name="base_joint" type="fixed">
-    <parent link="base_footprint"/>
-    <child link="base_link"/>
+  <xacro:arg name="color" default="red"/>
+  <xacro:property name="color" value="$(arg prefix)"/>
+  <link name="${color}_base_footprint"/>
+  <joint name="${color}_base_joint" type="fixed">
+    <parent link="${color}_base_footprint"/>
+    <child link="${color}_base_link"/>
     <origin xyz="0.0 0.0 0.010" rpy="0 0 0"/>
   </joint>
-  <link name="base_link">
+  <link name="${color}_base_link">
     <visual>
       <origin xyz="-0.032 0 0.0" rpy="0 0 0"/>
@@ -18,5 +20,5 @@
         <mesh filename="package://nuturtle_description/meshes/burger_base.stl" scale="0.001 0.001 0.001"/>
       </geometry>
-      <material name="light_black"/>
+      <material name="${color}"/>
     </visual>
     <collision>
@@ -34,11 +36,11 @@
     </inertial>
   </link>
-  <joint name="wheel_left_joint" type="continuous">
-    <parent link="base_link"/>
-    <child link="wheel_left_link"/>
+  <joint name="${color}_wheel_left_joint" type="continuous">
+    <parent link="${color}_base_link"/>
+    <child link="${color}_wheel_left_link"/>
     <origin xyz="0.0 ${track_width/2} 0.023" rpy="-1.57 0 0"/>
     <axis xyz="0 0 1"/>
   </joint>
-  <link name="wheel_left_link">
+  <link name="${color}_wheel_left_link">
     <visual>
       <origin xyz="0 0 0" rpy="1.57 0 0"/>
@@ -46,5 +48,5 @@
         <mesh filename="package://nuturtle_description/meshes/left_tire.stl" scale="0.001 0.001 0.001"/>
       </geometry>
-      <material name="dark"/>
+      <material name="${color}"/>
     </visual>
     <collision>
@@ -62,11 +64,11 @@
       </inertial>
   </link>
-  <joint name="wheel_right_joint" type="continuous">
-    <parent link="base_link"/>
-    <child link="wheel_right_link"/>
+  <joint name="${color}_wheel_right_joint" type="continuous">
+    <parent link="${color}_base_link"/>
+    <child link="${color}_wheel_right_link"/>
     <origin xyz="0.0 ${-track_width/2} 0.023" rpy="-1.57 0 0"/>
     <axis xyz="0 0 1"/>
   </joint>
-  <link name="wheel_right_link">
+  <link name="${color}_wheel_right_link">
     <visual>
       <origin xyz="0 0 0" rpy="1.57 0 0"/>
@@ -74,5 +76,5 @@
         <mesh filename="package://nuturtle_description/meshes/right_tire.stl" scale="0.001 0.001 0.001"/>
       </geometry>
-      <material name="dark"/>
+      <material name="${color}"/>
     </visual>
     <collision>
@@ -90,10 +92,10 @@
       </inertial>
   </link>
-  <joint name="caster_back_joint" type="fixed">
-    <parent link="base_link"/>
-    <child link="caster_back_link"/>
+  <joint name="${color}_caster_back_joint" type="fixed">
+    <parent link="${color}_base_link"/>
+    <child link="${color}_caster_back_link"/>
     <origin xyz="-0.081 0 -0.004" rpy="-1.57 0 0"/>
   </joint>
-  <link name="caster_back_link">
+  <link name="${color}_caster_back_link">
     <collision>
       <origin xyz="0 0.001 0" rpy="0 0 0"/>
@@ -110,16 +112,16 @@
     </inertial>
   </link>
-  <joint name="imu_joint" type="fixed">
-    <parent link="base_link"/>
-    <child link="imu_link"/>
+  <joint name="${color}_imu_joint" type="fixed">
+    <parent link="${color}_base_link"/>
+    <child link="${color}_imu_link"/>
     <origin xyz="-0.032 0 0.068" rpy="0 0 0"/>
   </joint>
-  <link name="imu_link"/>
-  <joint name="scan_joint" type="fixed">
-    <parent link="base_link"/>
-    <child link="base_scan"/>
+  <link name="${color}_imu_link"/>
+  <joint name="${color}_scan_joint" type="fixed">
+    <parent link="${color}_base_link"/>
+    <child link="${color}_base_scan"/>
     <origin xyz="-0.032 0 0.172" rpy="0 0 0"/>
   </joint>
-  <link name="base_scan">
+  <link name="${color}_base_scan">
     <visual>
       <origin xyz="0 0 0.0" rpy="0 0 0"/>
@@ -127,5 +129,5 @@
         <mesh filename="package://nuturtle_description/meshes/lds.stl" scale="0.001 0.001 0.001"/>
       </geometry>
-      <material name="dark"/>
+      <material name="${color}"/>
     </visual>
     <collision>

Commit message: Task A.8 done

File: nuturtle_description/urdf/turtlebot3_burger.urdf.xacro (robot description, xacro)
@@ -6,4 +6,5 @@
   <xacro:property name="wheel_radius" value="${param['wheel_radius']}" />
   <xacro:property name="track_width" value="${param['track_width']}" />
+  <xacro:property name="collision_radius" value="${param['collision_radius']}"/>
   <xacro:arg name="color" default="red"/>
   <xacro:property name="color" value="$(arg prefix)"/>
@@ -25,5 +26,10 @@
       <origin xyz="-0.032 0 0.070" rpy="0 0 0"/>
       <geometry>
+      <xacro:if value="${collision_radius != 0}">
+        <cylinder length="0.170" radius="${collision_radius}"/>
+      </xacro:if>
+      <xacro:if value="${collision_radius==0}">
         <box size="0.140 0.140 0.143"/>
+      </xacro:if>
       </geometry>
     </collision>
